File: PCB/radiopcb/radiopcb.kicad_sch (KiCad schematic)
At the start: 20 parts, among them CN1 PJ-3200, J1 Conn_01x02, J2 Conn_01x02, SW1 PWR, U1 XIAO-RP2040-DIP, U2 RDA5807MRRD-102V2.0, U3 TDA2822NBD

Commit message: pcb file changes
Parts:
- J2: footprint Connector:FanPinHeader_1x03_P2.54mm_Vertical -> Connector_PinHeader_2.54mm:PinHeader_1x02_P2.54mm_Vertical
- RV1, RV2: footprint Connector:FanPinHeader_1x03_P2.54mm_Vertical -> Connector_PinHeader_2.54mm:PinHeader_1x03_P2.54mm_Vertical
- U1: footprint Module:MOUDLE14P-XIAO-DIP-SMD -> Static:XIAO-RP2040-DIP
Connections:
- net L-OUT is gone; now on net L_OUT: U2.7 (L-OUT)
- net R-OUT is gone; now on net R_OUT: U2.8 (R-OUT)
- net GND: now also U2.10 (ANT); no longer CN1.4
- net at CN1.3: no longer U2.10 (ANT)
- no-connect marks 1 -> 0
Other:
- moved on the sheet: CN1
Changed lines of the file:
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@@
 		(color 0 0 0 0)
 	)
-	(no_connect
-		(at 163.83 104.14)
-	)
 	(wire
 		(pts
@@
 	(wire
 		(pts
-			(xy 163.83 107.95) (xy 163.83 106.68)
+			(xy 163.83 101.6) (xy 163.83 107.95)
 		)
 		(stroke
@@
 		)
 	)
-	(label "R-OUT"
+	(label "R_OUT"
 		(at 140.97 106.68 0)
 		(effects
@@
 		)
 	)
-	(label "L-OUT"
+	(label "L_OUT"
 		(at 140.97 109.22 0)
 		(effects
@@
 			)
 		)
-		(property "Footprint" "Connector:FanPinHeader_1x03_P2.54mm_Vertical"
+		(property "Footprint" "Connector_PinHeader_2.54mm:PinHeader_1x03_P2.54mm_Vertical"
 			(at 53.34 67.31 0)
 			(hide yes)
@@
 			)
 		)
-		(property "Footprint" "Connector:FanPinHeader_1x03_P2.54mm_Vertical"
+		(property "Footprint" "Connector_PinHeader_2.54mm:PinHeader_1x03_P2.54mm_Vertical"
 			(at 53.34 50.8 0)
 			(hide yes)
@@
 			)
 		)
-		(property "Footprint" "Connector:FanPinHeader_1x03_P2.54mm_Vertical"
+		(property "Footprint" "Connector_PinHeader_2.54mm:PinHeader_1x02_P2.54mm_Vertical"
 			(at 213.36 109.22 0)
 			(hide yes)
@@
 			)
 		)
-		(property "Footprint" "Module:MOUDLE14P-XIAO-DIP-SMD"
+		(property "Footprint" "Static:XIAO-RP2040-DIP"
 			(at 56.388 123.698 0)
 			(hide yes)
@@
 	(symbol
 		(lib_id "Static_Symbol_Library:PJ-3200")
-		(at 170.18 102.87 0)
-		(mirror y)
+		(at 170.18 102.87 90)
+		(mirror x)
 		(unit 1)
 		(body_style 1)
@@
 		(fields_autoplaced yes)
 		(property "Reference" "CN1"
-			(at 177.8 102.8699 0)
+			(at 175.26 99.4399 90)
 			(show_name no)
 			(do_not_autoplace no)
@@
 		)
 		(property "Value" "PJ-3200"
-			(at 177.8 105.4099 0)
+			(at 175.26 101.9799 90)
 			(show_name no)
 			(do_not_autoplace no)
@@
 		)
 		(property "Footprint" "Static:AUDIO-TH_PJ-3200"
-			(at 170.18 114.3 0)
+			(at 181.61 102.87 0)
 			(hide yes)
 			(show_name no)
@@
 		)
 		(property "Datasheet" "https://www.lcsc.com/datasheet/C2689690.pdf"
-			(at 170.18 116.84 0)
+			(at 184.15 102.87 0)
 			(hide yes)
 			(show_name no)
@@
 		)
 		(property "Manufacturer" "XKB Connection(中国星坤)"
-			(at 170.18 119.38 0)
+			(at 186.69 102.87 0)
 			(hide yes)
 			(show_name no)
@@
 		)
 		(property "MPN" "PJ-3200"
-			(at 170.18 121.92 0)
+			(at 189.23 102.87 0)
 			(hide yes)
 			(show_name no)
@@
 		)
 		(property "LCSC Part" "C2689690"
-			(at 170.18 124.46 0)
+			(at 191.77 102.87 0)
 			(hide yes)
 			(show_name no)
